File: layout/tweety.sch (EAGLE design)
At the start: 15 parts, among them IC2 MS563702BA03, J1 AVR_SPI_PRG_62X3_LOCK, U1 ATTINY88-MU

Commit message: initial layout
Parts:
- removed BAT1: BAT-HLD-001, vario_spc:CR2032
- removed J1: AVR_SPI_PRG_62X3_LOCK, SparkFun:AVR_SPI_PRG_62X3_LOCK
- removed K1: (no value), Seeed-OPL-Switch:SMD-SWITCH-TACTILE-SPST-NO(4P-D6.0MM)
- added JP1: AVR-ISP-6VERT, avr-7:AVR-ISP-6VERT
- added L2: sdr0503 10-15mH, vario_spc:SDR0503
- added P1: CR2450, vario_spc:CR2450
- added SJ1: SOLDERJUMPERTRACE, SparkFun:SOLDERJUMPERTRACE
- added SW1: (no value), EAGLE-TACT_SWITCHES-rev1:4301X20858X6
- added TP1, TP2: PTR1B2,54, testpad:PTR1B2,54
- added U$1: BSS138, m-pad-1.5:BSS138
- R4: value 4k7 -> 100k
Connections:
- new net N$3: L2.P$1, TP2.TP, U$1.D
- new net N$4: SJ1.2, U1.(PCINT0/CLKO/ICP1)_PB0
- new net PIEZO: U$1.G, U1.(PCINT1/OC1A)_PB1
- new net VPP: C1.1, L2.P$2, P1.P2, TP1.TP
- net GND: now also JP1.6, P1.N, SJ1.1, SW1.1, SW1.2, U$1.S; no longer BAT1.N, J1.6, K1.B0, K1.B1
- net MISO: now also JP1.1; no longer J1.1
- net MOSI: now also JP1.4; no longer J1.4
- net N$2: now also SW1.3, SW1.4; no longer K1.A0, K1.A1
- net RESET: now also JP1.5; no longer J1.5
- net SCK: now also JP1.3; no longer J1.3
- net VBAT: now also JP1.2, P1.P1; no longer BAT1.P1, BAT1.P2, C1.1, J1.2
- net VCC: now also U1.PC0_(ADC0/PCINT8)
Other:
- note added: "DISABLE PULLUP after evaluation"
- note added: "TEST"
- note added: "both: TBR?"
- note added: "todo jumper"
- note removed: "jumper todo"
- note removed: "piezo todo"
- note removed: "vcc todo!"
- moved on the sheet: C4

Commit message: v0.2
Parts:
- removed P1: CR2450, vario_spc:CR2450
- removed TP1, TP2: PTR1B2,54, testpad:PTR1B2,54
- added BAT1: KEYSTONE3008, vario_spc:KEYSTONE3008
- added C5: 10u, rcl-2:C-EUC0805
- added P2: PKLCS1212E2400, vario_spc:PKLCS1212E2400
- L2: value sdr0503 10-15mH -> 4m7-15m
Connections:
- new net N$5: U1.(PCINT2/SS/OC1B)_PB2
- net GND: now also BAT1.N, C5.2; no longer P1.N
- net N$2: no longer SW1.4
- net N$3: now also P2.P$+; no longer TP2.TP
- net VBAT: now also BAT1.P1; no longer P1.P1
- net VPP: now also BAT1.P2, C5.1, P2.P$-; no longer P1.P2, TP1.TP
Other:
- note removed: "TEST"
Changed lines of the file:
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@@
 <part name="GND10" library="supply1" deviceset="GND" device=""/>
 <part name="V10" library="supply" deviceset="VBAT" device=""/>
-<part name="P1" library="vario_spc" deviceset="CR2450" device=""/>
 <part name="SW1" library="EAGLE-TACT_SWITCHES-rev1" deviceset="4301X20858X6" device=""/>
 <part name="JP1" library="avr-7" deviceset="AVR-ISP-6" device="VERT"/>
@@
 <part name="U$1" library="m-pad-1.5" deviceset="BSS138" device=""/>
 <part name="GND11" library="supply1" deviceset="GND" device=""/>
-<part name="L2" library="vario_spc" deviceset="SDR0503" device="" value="sdr0503 10-15mH"/>
 <part name="V2" library="supply" deviceset="VPP" device=""/>
 <part name="V12" library="supply" deviceset="VPP" device=""/>
@@
 <part name="SJ1" library="SparkFun" deviceset="SOLDERJUMPER" device="TRACE"/>
 <part name="GND12" library="supply1" deviceset="GND" device=""/>
-<part name="TP1" library="testpad" deviceset="PTR1" device="B2,54"/>
-<part name="TP2" library="testpad" deviceset="PTR1" device="B2,54"/>
+<part name="P2" library="vario_spc" deviceset="PKLCS1212E2400" device=""/>
+<part name="BAT1" library="vario_spc" deviceset="KEYSTONE3008" device=""/>
+<part name="L2" library="vario_spc" deviceset="SDR0503" device="" value="4m7-15m"/>
+<part name="C5" library="rcl-2" deviceset="C-EU" device="C0805" value="10u"/>
+<part name="GND13" library="supply1" deviceset="GND" device=""/>
+<part name="V14" library="supply" deviceset="VPP" device=""/>
 </parts>
 <sheets>
@@
 <text x="10.16" y="60.96" size="1.778" layer="91">DISABLE PULLUP
 after evaluation</text>
-<text x="93.98" y="149.86" size="1.778" layer="94">TEST</text>
 </plain>
 <instances>
@@
 <instance part="GND10" gate="1" x="17.78" y="73.66"/>
 <instance part="V10" gate="G$1" x="17.78" y="96.52"/>
-<instance part="P1" gate="G$1" x="22.86" y="154.94"/>
 <instance part="SW1" gate="G$1" x="161.29" y="64.77" rot="R270"/>
 <instance part="JP1" gate="G$1" x="226.06" y="50.8"/>
@@
 <instance part="U$1" gate="G$1" x="83.82" y="132.08"/>
 <instance part="GND11" gate="1" x="86.36" y="119.38"/>
-<instance part="L2" gate="G$1" x="86.36" y="149.86" rot="R90"/>
 <instance part="V2" gate="G$1" x="25.4" y="167.64"/>
 <instance part="V12" gate="G$1" x="33.02" y="167.64"/>
@@
 <instance part="SJ1" gate="1" x="25.4" y="55.88"/>
 <instance part="GND12" gate="1" x="15.24" y="15.24"/>
-<instance part="TP1" gate="G$1" x="93.98" y="157.48" rot="R90"/>
-<instance part="TP2" gate="G$1" x="93.98" y="142.24" rot="R90"/>
+<instance part="P2" gate="G$1" x="101.6" y="149.86" rot="MR180"/>
+<instance part="BAT1" gate="G$1" x="22.86" y="154.94"/>
+<instance part="L2" gate="G$1" x="86.36" y="149.86" rot="R90"/>
+<instance part="C5" gate="G$1" x="40.64" y="157.48"/>
+<instance part="GND13" gate="1" x="40.64" y="144.78"/>
+<instance part="V14" gate="G$1" x="40.64" y="167.64"/>
 </instances>
 <busses>
@@
 <pinref part="GND1" gate="1" pin="GND"/>
 <wire x1="22.86" y1="149.86" x2="22.86" y2="147.32" width="0.1524" layer="91"/>
-<pinref part="P1" gate="G$1" pin="N"/>
+<pinref part="BAT1" gate="G$1" pin="N"/>
 </segment>
 <segment>
@@
 <wire x1="15.24" y1="55.88" x2="15.24" y2="17.78" width="0.1524" layer="91"/>
 </segment>
+<segment>
+<pinref part="C5" gate="G$1" pin="2"/>
+<pinref part="GND13" gate="1" pin="GND"/>
+<wire x1="40.64" y1="147.32" x2="40.64" y2="152.4" width="0.1524" layer="91"/>
+</segment>
 </net>
 <net name="VBAT" class="0">
@@
 <pinref part="V1" gate="G$1" pin="VBAT"/>
 <wire x1="20.32" y1="160.02" x2="20.32" y2="165.1" width="0.1524" layer="91"/>
-<pinref part="P1" gate="G$1" pin="P1"/>
+<pinref part="BAT1" gate="G$1" pin="P1"/>
 </segment>
 <segment>
@@
 <pinref part="U1" gate="A" pin="PD2_(INT0/PCINT18)"/>
 <pinref part="R4" gate="G$1" pin="1"/>
-<wire x1="157.48" y1="73.66" x2="154.94" y2="73.66" width="0.1524" layer="91"/>
-<wire x1="154.94" y1="73.66" x2="142.24" y2="73.66" width="0.1524" layer="91"/>
+<wire x1="157.48" y1="73.66" x2="142.24" y2="73.66" width="0.1524" layer="91"/>
 <wire x1="142.24" y1="73.66" x2="132.08" y2="73.66" width="0.1524" layer="91"/>
 <wire x1="142.24" y1="73.66" x2="142.24" y2="81.28" width="0.1524" layer="91"/>
@@
 <pinref part="SW1" gate="G$1" pin="3"/>
 <wire x1="157.48" y1="73.66" x2="157.48" y2="71.12" width="0.1524" layer="91"/>
-<pinref part="SW1" gate="G$1" pin="4"/>
-<wire x1="157.48" y1="58.42" x2="157.48" y2="55.88" width="0.1524" layer="91"/>
-<wire x1="157.48" y1="55.88" x2="154.94" y2="55.88" width="0.1524" layer="91"/>
-<wire x1="154.94" y1="55.88" x2="154.94" y2="73.66" width="0.1524" layer="91"/>
-<junction x="154.94" y="73.66"/>
 </segment>
 </net>
@@
 <net name="VPP" class="0">
 <segment>
-<pinref part="P1" gate="G$1" pin="P2"/>
 <pinref part="V2" gate="G$1" pin="VPP"/>
 <wire x1="25.4" y1="165.1" x2="25.4" y2="160.02" width="0.1524" layer="91"/>
+<pinref part="BAT1" gate="G$1" pin="P2"/>
 </segment>
 <segment>
@@
 </segment>
 <segment>
-<pinref part="L2" gate="G$1" pin="P$2"/>
 <pinref part="V13" gate="G$1" pin="VPP"/>
 <wire x1="86.36" y1="165.1" x2="86.36" y2="157.48" width="0.1524" layer="91"/>
-<pinref part="TP1" gate="G$1" pin="TP"/>
 <wire x1="86.36" y1="157.48" x2="86.36" y2="154.94" width="0.1524" layer="91"/>
-<wire x1="91.44" y1="157.48" x2="86.36" y2="157.48" width="0.1524" layer="91"/>
 <junction x="86.36" y="157.48"/>
+<wire x1="96.52" y1="152.4" x2="96.52" y2="157.48" width="0.1524" layer="91"/>
+<wire x1="96.52" y1="157.48" x2="86.36" y2="157.48" width="0.1524" layer="91"/>
+<pinref part="L2" gate="G$1" pin="P$2"/>
+<pinref part="P2" gate="G$1" pin="P$-"/>
+<wire x1="96.52" y1="152.4" x2="99.06" y2="152.4" width="0.1524" layer="91"/>
+</segment>
+<segment>
+<pinref part="C5" gate="G$1" pin="1"/>
+<pinref part="V14" gate="G$1" pin="VPP"/>
+<wire x1="40.64" y1="165.1" x2="40.64" y2="160.02" width="0.1524" layer="91"/>
 </segment>
 </net>
 <net name="N$3" class="0">
 <segment>
-<pinref part="L2" gate="G$1" pin="P$1"/>
 <pinref part="U$1" gate="G$1" pin="D"/>
 <wire x1="86.36" y1="144.78" x2="86.36" y2="142.24" width="0.1524" layer="91"/>
-<pinref part="TP2" gate="G$1" pin="TP"/>
 <wire x1="86.36" y1="142.24" x2="86.36" y2="137.16" width="0.1524" layer="91"/>
-<wire x1="91.44" y1="142.24" x2="86.36" y2="142.24" width="0.1524" layer="91"/>
 <junction x="86.36" y="142.24"/>
+<wire x1="86.36" y1="142.24" x2="96.52" y2="142.24" width="0.1524" layer="91"/>
+<wire x1="96.52" y1="142.24" x2="96.52" y2="147.32" width="0.1524" layer="91"/>
+<pinref part="L2" gate="G$1" pin="P$1"/>
+<pinref part="P2" gate="G$1" pin="P$+"/>
+<wire x1="96.52" y1="147.32" x2="99.06" y2="147.32" width="0.1524" layer="91"/>
 </segment>
 </net>
@@
 </segment>
 </net>
+<net name="N$5" class="0">
+<segment>
+<pinref part="U1" gate="A" pin="(PCINT2/SS/OC1B)_PB2"/>
+<wire x1="35.56" y1="50.8" x2="30.48" y2="50.8" width="0.1524" layer="91"/>
+</segment>
+</net>

Commit message: mount added
Other:
- note added: "todo: pull down?"
Changed lines of the file:
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@@
 <text x="10.16" y="60.96" size="1.778" layer="91">DISABLE PULLUP
 after evaluation</text>
+<text x="55.88" y="124.46" size="1.778" layer="91">todo: pull down?</text>
 </plain>
 <instances>

Commit message: v1.0
Parts:
- removed C5: 10u, rcl-2:C-EUC0805
- removed SJ1: SOLDERJUMPERTRACE, SparkFun:SOLDERJUMPERTRACE
- added GOLD_ORB_SM1: OSHWLOGO_GOLD_ORB_MED, bfl:OSHWLOGO_GOLD_ORB_MED
- C1: value 10u -> 22uF (Mouser 15Cent); device rcl-2:C-EUC0805 -> cap-master:CP-3528-21R
- L2: value 4m7-15m -> 3m3
- R1: value 4k7 -> NC
- R4: value 100k -> NC
Connections:
- removed net N$4: SJ1.2, U1.(PCINT0/CLKO/ICP1)_PB0
- removed net N$5: U1.(PCINT2/SS/OC1B)_PB2
- net GND: now also C1.-; no longer C1.2, C5.2, SJ1.1
- net VPP: now also C1.+; no longer C1.1, C5.1
Other:
- note removed: "DISABLE PULLUP after evaluation"
- note removed: "both: TBR?"
- note removed: "todo jumper"
- note removed: "todo: pull down?"
- moved on the sheet: BAT1
Changed lines of the file:
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@@
 <part name="V1" library="supply" deviceset="VBAT" device=""/>
 <part name="GND1" library="supply1" deviceset="GND" device=""/>
-<part name="C1" library="rcl-2" deviceset="C-EU" device="C0805" value="10u"/>
 <part name="GND2" library="supply1" deviceset="GND" device=""/>
 <part name="V3" library="supply" deviceset="VBAT" device=""/>
 <part name="GND3" library="supply1" deviceset="GND" device=""/>
-<part name="R1" library="rcl-2" deviceset="R-EU_" device="R0603" value="4k7"/>
+<part name="R1" library="rcl-2" deviceset="R-EU_" device="R0603" value="NC"/>
 <part name="V4" library="supply" deviceset="VBAT" device=""/>
 <part name="V5" library="supply" deviceset="VBAT" device=""/>
@@
 <part name="V7" library="supply" deviceset="VCC" device=""/>
 <part name="V8" library="supply" deviceset="VCC" device=""/>
-<part name="R4" library="rcl-2" deviceset="R-EU_" device="R0603" value="100k"/>
+<part name="R4" library="rcl-2" deviceset="R-EU_" device="R0603" value="NC"/>
 <part name="V9" library="supply" deviceset="VBAT" device=""/>
 <part name="GND9" library="supply1" deviceset="GND" device=""/>
@@
 <part name="V12" library="supply" deviceset="VPP" device=""/>
 <part name="V13" library="supply" deviceset="VPP" device=""/>
-<part name="SJ1" library="SparkFun" deviceset="SOLDERJUMPER" device="TRACE"/>
-<part name="GND12" library="supply1" deviceset="GND" device=""/>
 <part name="P2" library="vario_spc" deviceset="PKLCS1212E2400" device=""/>
 <part name="BAT1" library="vario_spc" deviceset="KEYSTONE3008" device=""/>
-<part name="L2" library="vario_spc" deviceset="SDR0503" device="" value="4m7-15m"/>
-<part name="C5" library="rcl-2" deviceset="C-EU" device="C0805" value="10u"/>
-<part name="GND13" library="supply1" deviceset="GND" device=""/>
-<part name="V14" library="supply" deviceset="VPP" device=""/>
+<part name="L2" library="vario_spc" deviceset="SDR0503" device="" value="3m3"/>
+<part name="C1" library="cap-master" deviceset="CP-" device="3528-21R" value="22uF (Mouser 15Cent)"/>
+<part name="GOLD_ORB_SM1" library="bfl" deviceset="OSHWLOGO" device="_GOLD_ORB_MED"/>
 </parts>
 <sheets>
 <sheet>
 <plain>
-<text x="114.3" y="86.36" size="1.778" layer="91">both: TBR?</text>
-<text x="25.4" y="114.3" size="1.778" layer="91">todo jumper</text>
-<text x="10.16" y="60.96" size="1.778" layer="91">DISABLE PULLUP
-after evaluation</text>
-<text x="55.88" y="124.46" size="1.778" layer="91">todo: pull down?</text>
 </plain>
 <instances>
@@
 <instance part="C35" gate="G$1" x="187.96" y="139.7"/>
 <instance part="L1" gate="G$1" x="180.34" y="152.4" rot="R90"/>
-<instance part="V1" gate="G$1" x="20.32" y="167.64"/>
-<instance part="GND1" gate="1" x="22.86" y="144.78"/>
-<instance part="C1" gate="G$1" x="33.02" y="157.48"/>
-<instance part="GND2" gate="1" x="33.02" y="144.78"/>
+<instance part="V1" gate="G$1" x="20.32" y="157.48"/>
+<instance part="GND1" gate="1" x="22.86" y="134.62"/>
+<instance part="GND2" gate="1" x="33.02" y="134.62"/>
 <instance part="V3" gate="G$1" x="33.02" y="96.52"/>
 <instance part="GND3" gate="1" x="33.02" y="15.24"/>
@@
 <instance part="U$1" gate="G$1" x="83.82" y="132.08"/>
 <instance part="GND11" gate="1" x="86.36" y="119.38"/>
-<instance part="V2" gate="G$1" x="25.4" y="167.64"/>
-<instance part="V12" gate="G$1" x="33.02" y="167.64"/>
+<instance part="V2" gate="G$1" x="25.4" y="157.48"/>
+<instance part="V12" gate="G$1" x="33.02" y="157.48"/>
 <instance part="V13" gate="G$1" x="86.36" y="167.64"/>
-<instance part="SJ1" gate="1" x="25.4" y="55.88"/>
-<instance part="GND12" gate="1" x="15.24" y="15.24"/>
 <instance part="P2" gate="G$1" x="101.6" y="149.86" rot="MR180"/>
-<instance part="BAT1" gate="G$1" x="22.86" y="154.94"/>
+<instance part="BAT1" gate="G$1" x="22.86" y="144.78"/>
 <instance part="L2" gate="G$1" x="86.36" y="149.86" rot="R90"/>
-<instance part="C5" gate="G$1" x="40.64" y="157.48"/>
-<instance part="GND13" gate="1" x="40.64" y="144.78"/>
-<instance part="V14" gate="G$1" x="40.64" y="167.64"/>
+<instance part="C1" gate="G$1" x="33.02" y="144.78" rot="R90"/>
+<instance part="GOLD_ORB_SM1" gate="G$1" x="187.96" y="15.24"/>
 </instances>
 <busses>
@@
 <segment>
 <pinref part="GND1" gate="1" pin="GND"/>
-<wire x1="22.86" y1="149.86" x2="22.86" y2="147.32" width="0.1524" layer="91"/>
+<wire x1="22.86" y1="139.7" x2="22.86" y2="137.16" width="0.1524" layer="91"/>
 <pinref part="BAT1" gate="G$1" pin="N"/>
 </segment>
 <segment>
-<pinref part="C1" gate="G$1" pin="2"/>
 <pinref part="GND2" gate="1" pin="GND"/>
-<wire x1="33.02" y1="147.32" x2="33.02" y2="152.4" width="0.1524" layer="91"/>
+<wire x1="33.02" y1="137.16" x2="33.02" y2="142.24" width="0.1524" layer="91"/>
+<pinref part="C1" gate="G$1" pin="-"/>
 </segment>
 <segment>
@@
 <wire x1="86.36" y1="121.92" x2="86.36" y2="127" width="0.1524" layer="91"/>
 </segment>
-<segment>
-<pinref part="SJ1" gate="1" pin="1"/>
-<pinref part="GND12" gate="1" pin="GND"/>
-<wire x1="20.32" y1="55.88" x2="15.24" y2="55.88" width="0.1524" layer="91"/>
-<wire x1="15.24" y1="55.88" x2="15.24" y2="17.78" width="0.1524" layer="91"/>
-</segment>
-<segment>
-<pinref part="C5" gate="G$1" pin="2"/>
-<pinref part="GND13" gate="1" pin="GND"/>
-<wire x1="40.64" y1="147.32" x2="40.64" y2="152.4" width="0.1524" layer="91"/>
-</segment>
 </net>
 <net name="VBAT" class="0">
 <segment>
 <pinref part="V1" gate="G$1" pin="VBAT"/>
-<wire x1="20.32" y1="160.02" x2="20.32" y2="165.1" width="0.1524" layer="91"/>
+<wire x1="20.32" y1="149.86" x2="20.32" y2="154.94" width="0.1524" layer="91"/>
 <pinref part="BAT1" gate="G$1" pin="P1"/>
 </segment>
@@
 <segment>
 <pinref part="V2" gate="G$1" pin="VPP"/>
-<wire x1="25.4" y1="165.1" x2="25.4" y2="160.02" width="0.1524" layer="91"/>
+<wire x1="25.4" y1="154.94" x2="25.4" y2="149.86" width="0.1524" layer="91"/>
 <pinref part="BAT1" gate="G$1" pin="P2"/>
 </segment>
 <segment>
-<pinref part="C1" gate="G$1" pin="1"/>
 <pinref part="V12" gate="G$1" pin="VPP"/>
-<wire x1="33.02" y1="165.1" x2="33.02" y2="160.02" width="0.1524" layer="91"/>
+<wire x1="33.02" y1="154.94" x2="33.02" y2="147.32" width="0.1524" layer="91"/>
+<pinref part="C1" gate="G$1" pin="+"/>
 </segment>
 <segment>
@@
 <wire x1="96.52" y1="152.4" x2="99.06" y2="152.4" width="0.1524" layer="91"/>
 </segment>
-<segment>
-<pinref part="C5" gate="G$1" pin="1"/>
-<pinref part="V14" gate="G$1" pin="VPP"/>
-<wire x1="40.64" y1="165.1" x2="40.64" y2="160.02" width="0.1524" layer="91"/>
-</segment>
 </net>
 <net name="N$3" class="0">
@@
 </segment>
 </net>
-<net name="N$4" class="0">
-<segment>
-<pinref part="U1" gate="A" pin="(PCINT0/CLKO/ICP1)_PB0"/>
-<pinref part="SJ1" gate="1" pin="2"/>
-<wire x1="30.48" y1="55.88" x2="35.56" y2="55.88" width="0.1524" layer="91"/>
-</segment>
-</net>
-<net name="N$5" class="0">
-<segment>
-<pinref part="U1" gate="A" pin="(PCINT2/SS/OC1B)_PB2"/>
-<wire x1="35.56" y1="50.8" x2="30.48" y2="50.8" width="0.1524" layer="91"/>
-</segment>
-</net>
 </nets>
 </sheet>
@@
 </schematic>
 </drawing>
-<compatibility>
-<note version="6.3" minversion="6.2.2" severity="warning">
-Since Version 6.2.2 text objects can contain more than one line,
-which will not be processed correctly with this version.
-</note>
-</compatibility>
 </eagle>
