File: layout/tweety.brd (EAGLE design)
At the start: 28 x 46 mm, 15 parts, among them IC2 MS563702BA03, J1 AVR_SPI_PRG_62X3_LOCK, U1 ATTINY88-MU

Commit message: initial layout
Parts:
- removed BAT1: BAT-HLD-001, vario_spc:CR2032
- removed J1: AVR_SPI_PRG_62X3_LOCK, SparkFun:2X3_LOCK
- removed K1: (no value), Seeed-OPL-Switch:SW4-SMD-6.0X6.0X5.0MM
- added JP1: AVR-ISP-6VERT, avr-7:AVR-ISP-6
- added L2: sdr0503 10-15mH, vario_spc:SDR0503
- added P1: CR2450, vario_spc:CR2450
- added SJ1: SOLDERJUMPERTRACE, SparkFun:SJ_2S-TRACE
- added SW1: (no value), EAGLE-TACT_SWITCHES-rev1:4301X20858X6
- added TP1, TP2: PTR1B2,54, testpad:B2,54
- added U$1: BSS138, m-pad-1.5:SOT23
- R4: value 4k7 -> 100k
- moved L1 37.8 mm to (2.00, 21.7), turned to 270 degrees
- moved C3 36.7 mm to (4.40, 22.7), turned to 0 degrees
- moved C35 34.5 mm to (4.40, 20.7), turned to 0 degrees
- moved R4 32.8 mm to (2.59, 25.9), turned to 90 degrees
- moved C2 32.3 mm to (4.40, 18.6), turned to 0 degrees
- moved R2 32.2 mm to (3.00, 12.3), turned to 270 degrees
- moved IC2 30.1 mm to (4.05, 15.8), turned to 0 degrees
- moved R3 29.2 mm to (5.03, 12.3), turned to 270 degrees
- moved R1 28.8 mm to (4.62, 25.9), turned to 90 degrees
- moved C1 21.1 mm to (25.8, 25.5), turned to 180 degrees
- moved U1 13.2 mm to (5.24, 7.57), turned to 90 degrees
- moved C4 13.1 mm to (6.75, 2.70), turned to 90 degrees
Connections:
- new net N$3: L2.P$1, TP2.TP, U$1.3
- new net N$4: SJ1.2, U1.12
- new net PIEZO: U$1.1, U1.13
- new net VPP: C1.1, L2.P$2, P1.P$2, TP1.TP
- net GND: now also JP1.6, P1.N, SJ1.1, SW1.1, SW1.2, U$1.2; no longer BAT1.N, J1.6, K1.2, K1.3
- net MISO: now also JP1.1; no longer J1.1
- net MOSI: now also JP1.4; no longer J1.4
- net N$2: now also SW1.3, SW1.4; no longer K1.1, K1.4
- net RESET: now also JP1.5; no longer J1.5
- net SCK: now also JP1.3; no longer J1.3
- net VBAT: now also JP1.2, P1.P$1; no longer BAT1.P1, BAT1.P2, C1.1, J1.2
- net VCC: now also U1.23
Routing:
- net GND: track 0.00 -> 135.9 mm, vias 0 -> 16
- net VBAT: track 0.00 -> 61.8 mm, vias 0 -> 3
- net N$2: track 0.00 -> 44.7 mm, vias 0 -> 2
- net VPP: track 0.00 -> 33.5 mm, vias 0 -> 2
- net RESET: track 0.00 -> 31.3 mm, vias 0 -> 2
- net N$3: track 0.00 -> 30.6 mm
- net PIEZO: track 0.00 -> 19.7 mm
- net VCC: track 0.00 -> 19.3 mm, vias 0 -> 2
- net N$4: track 0.00 -> 19.0 mm
- net SCL: track 0.00 -> 13.5 mm
- net MOSI: track 0.00 -> 12.9 mm
- net SCK: track 0.00 -> 9.90 mm
- net SDA: track 0.00 -> 9.68 mm
- net MISO: track 0.00 -> 7.89 mm
- net N$1: track 0.00 -> 5.67 mm
- added copper zone on layer 1, net GND
- added copper zone on layer 16, net GND
- added copper zone on layer 1, net N$3
- added copper zone on layer 1, net VPP
Other:
- board text added: "close gronund loop"
- board text added: "height 6mm"
- board text added: "tweety v0.1"

Commit message: v0.2
Parts:
- removed P1: CR2450, vario_spc:CR2450
- removed TP1, TP2: PTR1B2,54, testpad:B2,54
- added BAT1: KEYSTONE3008, vario_spc:KEYSTONE3008
- added C5: 10u, rcl-2:C0805
- added P2: PKLCS1212E2400, vario_spc:PKLCS1212
- L2: value sdr0503 10-15mH -> 4m7-15m
- moved R1 22.5 mm to (17.9, 7.80), turned to 0 degrees
- moved R4 16.7 mm to (19.2, 27.9)
- moved C3 14.3 mm to (16.3, 30.6)
- moved R3 14.3 mm to (16.9, 20.2)
- moved C2 14.3 mm to (16.3, 26.5)
- moved C35 14.3 mm to (16.3, 28.6)
- moved C4 14.3 mm to (18.7, 10.6)
- moved L1 14.3 mm to (13.9, 29.6)
- moved R2 14.3 mm to (14.9, 20.2)
- moved U1 14.3 mm to (17.1, 15.5)
- moved IC2 14.3 mm to (15.9, 23.7)
- moved SW1 12.9 mm to (26.6, 22.3)
- moved C1 12.4 mm to (38.2, 26.0)
- moved JP1 12.3 mm to (26.6, 20.3)
- moved L2 12.1 mm to (37.8, 19.7)
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Connections:
- new net N$5: U1.14
- net GND: now also BAT1.N, C5.2; no longer P1.N
- net N$2: no longer SW1.4
- net N$3: now also P2.P$+; no longer TP2.TP
- net VBAT: now also BAT1.P$3; no longer P1.P$1
- net VPP: now also BAT1.P$4, C5.1, P2.P$-; no longer P1.P$2, TP1.TP
Routing:
- net VBAT: track 61.8 -> 84.1 mm, vias 3 -> 4
- net N$2: track 44.7 -> 23.3 mm
- net GND: track 135.9 -> 122.9 mm, vias 16 -> 40
- net N$4: track 19.0 -> 8.52 mm, vias 0 -> 1
- net N$3: track 30.6 -> 21.7 mm
- net VPP: track 33.5 -> 27.7 mm
- net PIEZO: track 19.7 -> 15.5 mm
- net RESET: track 31.3 -> 27.9 mm, vias 2 -> 3
- net SCK: track 9.90 -> 7.73 mm
- net MOSI: track 12.9 -> 10.9 mm
- net MISO: track 7.89 -> 5.90 mm
- net VCC: track 19.3 -> 20.7 mm
- removed copper zone on layer 1, net N$3
- removed copper zone on layer 1, net VPP
Other:
- board size 28 x 46 mm -> 28.4 x 50 mm
- board text added: "Tweety v0.2"
- board text removed: "PCB thickness: 0.8mm"
- board text removed: "close gronund loop"
- board text removed: "height 6mm"
- board text removed: "tweety v0.1"

Commit message: v1.0
Parts:
- removed C5: 10u, rcl-2:C0805
- removed SJ1: SOLDERJUMPERTRACE, SparkFun:SJ_2S-TRACE
- added GOLD_ORB_SM1: OSHWLOGO_GOLD_ORB_MED, bfl:OSHW1
- C1: value 10u -> 22uF (Mouser 15Cent); device rcl-2:C0805 -> cap-master:3528-21R/T
- L2: value 4m7-15m -> 3m3
- R1: value 4k7 -> NC
- R4: value 100k -> NC
- moved C1 1.07 mm to (37.7, 25.1), turned to 0 degrees
- moved L2 0.25 mm to (37.8, 20.0)
- moved U$1 0.10 mm to (36.1, 15.0)
Connections:
- removed net N$4: SJ1.2, U1.12
- removed net N$5: U1.14
- net GND: now also C1.-; no longer C1.2, C5.2, SJ1.1
- net VPP: now also C1.+; no longer C1.1, C5.1
Routing:
- net N$4: track 8.52 -> 0.00 mm, vias 1 -> 0
- net GND: track 122.9 -> 115.8 mm, vias 40 -> 44
Other:
- board text added: "Tweety v1.0"
- board text removed: "Tweety v0.2"

Commit message: layout optimized
Routing:
- net VCC: track 20.7 -> 24.5 mm
- net GND: vias 44 -> 45
Other:
- board text added: "Tweety v1.1"
- board text removed: "Tweety v1.0"
Changed lines of the file:
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@@
 <?xml version="1.0" encoding="utf-8"?>
 <!DOCTYPE eagle SYSTEM "eagle.dtd">
-<eagle version="7.2.0">
+<eagle version="7.7.0">
 <drawing>
 <settings>
@@
 <setting verticaltext="up"/>
 </settings>
-<grid distance="10" unitdist="mil" unit="mil" style="lines" multiple="1" display="yes" altdistance="0.025" altunitdist="inch" altunit="inch"/>
+<grid distance="2" unitdist="mil" unit="mm" style="lines" multiple="1" display="yes" altdistance="0.025" altunitdist="inch" altunit="inch"/>
 <layers>
 <layer number="1" name="Top" color="4" fill="1" visible="yes" active="yes"/>
@@
 <board>
 <plain>
-<hole x="37.6" y="51.1" drill="3"/>
-<hole x="37.6" y="10.5" drill="3"/>
-<hole x="15.6" y="10.5" drill="3"/>
+<hole x="37.6" y="51.1" drill="3.1"/>
+<hole x="37.6" y="10.5" drill="3.1"/>
+<hole x="15.6" y="10.5" drill="3.1"/>
 <wire x1="25" y1="2" x2="32.4" y2="2" width="0.1" layer="37"/>
-<text x="31.6612" y="49.9116" size="1.27" layer="16" font="vector" ratio="17" rot="MR0">Tweety v1.0</text>
+<text x="31.6612" y="49.9116" size="1.27" layer="16" font="vector" ratio="17" rot="MR0">Tweety v1.1</text>
 <wire x1="26.6" y1="53.8" x2="26.6" y2="55.9" width="0.01" layer="37"/>
 <wire x1="26.6" y1="55.9" x2="26.6" y2="56.8" width="0.01" layer="37"/>
@@
 <wire x1="17.394" y1="12.9554" x2="17.394" y2="12.5208" width="0.3048" layer="1"/>
 <wire x1="33.528" y1="24.892" x2="36.068" y2="24.892" width="0.508" layer="1"/>
+<via x="20.982" y="22.6234" extent="1-16" drill="0.3048"/>
 </signal>
 <signal name="VBAT">
@@
 <wire x1="14.9114" y1="48.6584" x2="14.9114" y2="32.6564" width="0.3048" layer="16"/>
 <via x="19.6612" y="9.771" extent="1-16" drill="0.3048"/>
-<wire x1="16.886" y1="12.9554" x2="16.886" y2="12.2922" width="0.3048" layer="1"/>
-<wire x1="16.886" y1="12.2922" x2="17.7816" y2="11.3966" width="0.3048" layer="1"/>
-<wire x1="17.7816" y1="11.3966" x2="17.7816" y2="10.6092" width="0.3048" layer="1"/>
-<wire x1="17.7816" y1="10.6092" x2="17.7816" y2="10.0758" width="0.3048" layer="1"/>
-<wire x1="17.7816" y1="10.0758" x2="18.1074" y2="9.75" width="0.3048" layer="1"/>
+<wire x1="16.886" y1="12.9554" x2="16.886" y2="12.343" width="0.3048" layer="1"/>
+<wire x1="16.886" y1="12.343" x2="17.8324" y2="11.3966" width="0.3048" layer="1"/>
+<wire x1="17.8324" y1="11.3966" x2="17.8324" y2="10.6092" width="0.3048" layer="1"/>
+<wire x1="17.8324" y1="10.6092" x2="17.8324" y2="10.025" width="0.3048" layer="1"/>
+<wire x1="17.8324" y1="10.025" x2="18.1074" y2="9.75" width="0.3048" layer="1"/>
 <wire x1="18.1074" y1="9.75" x2="18.6524" y2="9.75" width="0.3048" layer="1"/>
 <wire x1="27.87" y1="17.7616" x2="26.7628" y2="16.6544" width="0.1524" layer="16"/>
@@
 <wire x1="20.4232" y1="16.6036" x2="18.061" y2="18.9658" width="0.1524" layer="16"/>
 <wire x1="19.712" y1="10.914" x2="19.4072" y2="10.6092" width="0.1524" layer="1"/>
-<wire x1="19.4072" y1="10.6092" x2="17.7816" y2="10.6092" width="0.1524" layer="1"/>
+<wire x1="19.4072" y1="10.6092" x2="17.8324" y2="10.6092" width="0.1524" layer="1"/>
 <wire x1="18.7632" y1="7.7996" x2="18.6524" y2="7.9104" width="0.1524" layer="1"/>
 <wire x1="18.6524" y1="7.9104" x2="18.6524" y2="9.75" width="0.1524" layer="1"/>
@@
 <wire x1="14.4796" y1="17.5688" x2="17.5356" y2="20.6248" width="0.1524" layer="16"/>
 <wire x1="17.0632" y1="7.7996" x2="17.4768" y2="8.2132" width="0.1524" layer="1"/>
-<wire x1="17.4768" y1="8.2132" x2="17.4768" y2="9.0598" width="0.1524" layer="1"/>
-<via x="17.4768" y="9.0598" extent="1-16" drill="0.3048"/>
-<wire x1="17.4768" y1="9.0598" x2="17.7054" y2="9.2884" width="0.1524" layer="16"/>
-<wire x1="17.7054" y1="9.2884" x2="17.7054" y2="11.3966" width="0.1524" layer="16"/>
-<wire x1="17.7054" y1="11.3966" x2="16.4862" y2="12.6158" width="0.1524" layer="16"/>
-<wire x1="16.4862" y1="12.6158" x2="14.886" y2="12.6158" width="0.1524" layer="16"/>
-<wire x1="14.886" y1="12.6158" x2="14.632" y2="12.3618" width="0.1524" layer="16"/>
-<wire x1="14.632" y1="12.3618" x2="14.0478" y2="12.3618" width="0.1524" layer="16"/>
-<wire x1="14.0478" y1="12.3618" x2="13.6922" y2="12.7174" width="0.1524" layer="16"/>
-<wire x1="13.6922" y1="12.7174" x2="13.6922" y2="13.2" width="0.1524" layer="16"/>
-<wire x1="13.6922" y1="13.2" x2="13.997" y2="13.5048" width="0.1524" layer="16"/>
-<wire x1="13.997" y1="13.5048" x2="13.997" y2="14.978" width="0.1524" layer="16"/>
+<wire x1="17.4768" y1="8.2132" x2="17.4768" y2="8.9582" width="0.1524" layer="1"/>
+<via x="17.4768" y="8.9582" extent="1-16" drill="0.3048"/>
+<wire x1="17.4768" y1="8.9582" x2="17.7562" y2="9.2376" width="0.1524" layer="16"/>
+<wire x1="17.7562" y1="9.2376" x2="17.7562" y2="11.3966" width="0.1524" layer="16"/>
+<wire x1="17.7562" y1="11.3966" x2="16.4862" y2="12.6666" width="0.1524" layer="16"/>
+<wire x1="16.4862" y1="12.6666" x2="14.8352" y2="12.6666" width="0.1524" layer="16"/>
+<wire x1="14.8352" y1="12.6666" x2="14.5304" y2="12.3618" width="0.1524" layer="16"/>
+<wire x1="14.5304" y1="12.3618" x2="13.997" y2="12.3618" width="0.1524" layer="16"/>
+<wire x1="13.997" y1="12.3618" x2="13.6414" y2="12.7174" width="0.1524" layer="16"/>
+<wire x1="13.6414" y1="12.7174" x2="13.6414" y2="13.2" width="0.1524" layer="16"/>
+<wire x1="13.6414" y1="13.2" x2="13.997" y2="13.5556" width="0.1524" layer="16"/>
+<wire x1="13.997" y1="13.5556" x2="13.997" y2="14.978" width="0.1524" layer="16"/>
 <wire x1="13.997" y1="14.978" x2="13.743" y2="15.232" width="0.1524" layer="16"/>
 <wire x1="17.5356" y1="20.6248" x2="21.2344" y2="20.6248" width="0.1524" layer="16"/>
@@
 <wire x1="15.8954" y1="20.2292" x2="15.902" y2="20.2358" width="0.3048" layer="1"/>
 <via x="15.902" y="20.2358" extent="1-16" drill="0.3048"/>
-<wire x1="15.902" y1="20.2358" x2="15.902" y2="29.7862" width="0.3048" layer="16"/>
-<wire x1="15.902" y1="29.7862" x2="14.1494" y2="31.5388" width="0.3048" layer="16"/>
 <via x="14.1494" y="31.5388" extent="1-16" drill="0.3048"/>
 <wire x1="13.8954" y1="30.4498" x2="13.9032" y2="30.442" width="0.3048" layer="1"/>
@@
 <wire x1="15.902" y1="20.2358" x2="16.0878" y2="20.2358" width="0.1524" layer="1"/>
 <wire x1="16.0878" y1="20.2358" x2="16.9292" y2="19.3944" width="0.1524" layer="1"/>
+<wire x1="14.1494" y1="31.5388" x2="19.3548" y2="26.3334" width="0.3048" layer="16"/>
+<wire x1="19.3548" y1="26.3334" x2="19.3548" y2="22.098" width="0.3048" layer="16"/>
+<wire x1="19.3548" y1="22.098" x2="18.3896" y2="21.1328" width="0.3048" layer="16"/>
+<wire x1="18.3896" y1="21.1328" x2="16.799" y2="21.1328" width="0.3048" layer="16"/>
+<wire x1="16.799" y1="21.1328" x2="15.902" y2="20.2358" width="0.3048" layer="16"/>
 </signal>
 <signal name="SDA">
@@
 <wire x1="18.3658" y1="21.0342" x2="18.3658" y2="26.2842" width="0.1524" layer="1"/>
 <wire x1="18.3658" y1="26.2842" x2="19.1562" y2="27.0746" width="0.1524" layer="1"/>
-<wire x1="14.6254" y1="13.7174" x2="14.3018" y2="13.3938" width="0.1524" layer="1"/>
-<wire x1="14.3018" y1="13.3938" x2="14.3018" y2="12.946" width="0.1524" layer="1"/>
-<via x="14.3018" y="12.946" extent="1-16" drill="0.3048"/>
-<wire x1="14.3018" y1="12.946" x2="14.8352" y2="13.4794" width="0.1524" layer="16"/>
+<wire x1="14.6254" y1="13.7174" x2="14.251" y2="13.343" width="0.1524" layer="1"/>
+<wire x1="14.251" y1="13.343" x2="14.251" y2="12.946" width="0.1524" layer="1"/>
+<via x="14.251" y="12.946" extent="1-16" drill="0.3048"/>
+<wire x1="14.251" y1="12.946" x2="14.8352" y2="13.4794" width="0.1524" layer="16"/>
 <wire x1="14.8352" y1="13.4794" x2="14.8352" y2="17.4418" width="0.1524" layer="16"/>
 <wire x1="14.8352" y1="17.4418" x2="17.7134" y2="20.32" width="0.1524" layer="16"/>
